Commit message: Fixed black material and joint limits

File: wsg_50_simulation/urdf/wsg_50.urdf.xacro (robot description, xacro)
@@ -45,5 +45,5 @@
   <!-- GRIPPER LEFT -->
   <joint name="${name}_base_joint_gripper_left" type="prismatic">
-     <limit lower="-0.055" upper="-0.0027" effort="1.0" velocity="1.0"/>
+     <limit lower="-0.055" upper="-0.0027" effort="1.0" velocity="0.42"/>
      <origin xyz="0 0 0" rpy="0 0 0" />      <!--origin xyz="-0.0067 0 0.049" rpy="0 0 0" /-->
      <parent link="${name}_base_link"/>
@@ -51,5 +51,5 @@
      <dynamics friction="100" damping="100" />
      <axis xyz="1 0 0"/>
-     <limit effort="100" velocity="100"/>
+     <!-- <limit effort="100" velocity="100"/> -->
   </joint>
   <transmission name="${name}_base_trans_left" type="pr2_mechanism_model/SimpleTransmission">
@@ -74,5 +74,5 @@
           </geometry>
           <material name="black">
-		<color rgba="0 0 0 0"/>
+		<color rgba="0 0 0 1"/>
       	  </material>
       </visual>
@@ -97,5 +97,5 @@
      <dynamics friction="100" damping="100" />
      <axis xyz="1 0 0"/>
-     <limit effort="100" velocity="100"/>
+     <!-- <limit effort="100" velocity="100"/> -->
   </joint>
   <link name="${name}_finger_left">
@@ -113,5 +113,5 @@
           </geometry>
           <material name="black">
-		<color rgba="0 0 0 0"/>
+		<color rgba="0 0 0 1"/>
       	  </material>
       </visual>
@@ -130,5 +130,5 @@
   <!-- GRIPPER RIGHT -->
   <joint name="${name}_base_joint_gripper_right" type="prismatic">
-     <limit lower="0.0027" upper="0.055" effort="1.0" velocity="1.0"/>
+     <limit lower="0.0027" upper="0.055" effort="1.0" velocity="0.42"/>
      <origin xyz="0 0 0" rpy="0 0 3.14159" />
      <parent link="${name}_base_link"/>
@@ -136,5 +136,5 @@
      <axis xyz="-1 0 0"/>
      <dynamics friction="100" damping="100" />
-     <limit effort="100" velocity="100"/>
+     <!-- <limit effort="100" velocity="100"/>-->
   </joint>
   <transmission name="${name}_base_trans_right" type="pr2_mechanism_model/SimpleTransmission">
@@ -159,5 +159,5 @@
           </geometry>
           <material name="black">
-		<color rgba="0 0 0 0"/>
+		<color rgba="0 0 0 1"/>
       	  </material>
       </visual>
@@ -198,5 +198,5 @@
           </geometry>
           <material name="black">
-		<color rgba="0 0 0 0"/>
+		<color rgba="0 0 0 1"/>
       	  </material>
       </visual>
